File: STM32F103_Hardware_Design.kicad_sch (KiCad schematic)
At the start: 28 parts, among them J1 USB_B_Micro, J2 Conn_01x04_Pin, J3 Conn_01x04_Pin, J4 Conn_01x04_Pin, SW1 SW_SPDT, U1 STM32F103C8T6, U2 AMS1117-3.3, Y2 16MHz

Commit message: PCB layout and component alignment done,\n usb port 3d model added
Parts:
- added H1, H2, H3, H4: MountingHole, MountingHole:MountingHole_2.2mm_M2, symbol Mechanical:MountingHole
- SW1: footprint Button_Switch_THT:SW_E-Switch_EG1224_SPDT_Angled -> Button_Switch_SMD:SW_SPDT_PCM12
Connections:
- net +3V3: now also J2.4 (Pin_4); no longer J2.1 (Pin_1)
- net GND: now also J2.1 (Pin_1); no longer J2.4 (Pin_4)
- net SWCLK: now also J2.2 (Pin_2); no longer J2.3 (Pin_3)
- net SWDIO: now also J2.3 (Pin_3); no longer J2.2 (Pin_2)
