File: STM32F103_Hardware_Design.kicad_pcb (KiCad board)
At the start: 2 copper layers, 40.1 x 32.1 mm, 32 parts, among them J1 USB_B_Micro, J2 Conn_01x04_Pin, J3 Conn_01x04_Pin, J4 Conn_01x04_Pin, SW1 SW_SPDT, U1 STM32F103C8T6, U2 AMS1117-3.3, Y2 16MHz

Commit message: PCB done
Parts:
- added REF**: KiCad-Logo2_8mm_SilkScreen, Symbol:KiCad-Logo2_8mm_SilkScreen, B.Cu at (149.1, 71.3)
- moved R1 13.3 mm to (132.5, 70.0), turned to 90 degrees
- moved Y2 1.22 mm to (136.4, 72.8)
- moved C11 1.22 mm to (139.3, 74.3)
- moved C10 1.16 mm to (139.2, 72.1)
- moved C6 0.90 mm to (141.2, 74.6), turned to 90 degrees
- moved C3 0.65 mm to (149.6, 80.0)
- moved R2 0.64 mm to (156.3, 71.6)
- moved C2 0.39 mm to (144.5, 67.1)
- moved J1 0.36 mm to (163.0, 72.1)
- moved C4 0.29 mm to (153.0, 71.0)
- moved C1 0.23 mm to (141.0, 70.2)
Connections:
- J1 pad 6: unconnected-(J1-Shield-Pad6) -> (no net)
Routing:
- net +3V3: track 0.00 -> 165.3 mm, vias 0 -> 2
- net GND: track 0.00 -> 32.0 mm, vias 0 -> 18
- net /boot0: track 0.00 -> 22.5 mm
- net /SWDIO: track 0.00 -> 14.1 mm
- net /I2C2_SCL: track 0.00 -> 13.5 mm
- net /USART1_RX: track 0.00 -> 13.0 mm
- net /I2C2_SDA: track 0.00 -> 11.3 mm
- net /USART1_TX: track 0.00 -> 11.1 mm
- net /USB_D+: track 0.00 -> 9.95 mm
- net /USB_D-: track 0.00 -> 9.92 mm
- net /SWCLK: track 0.00 -> 9.81 mm
- net /NRST: track 0.00 -> 8.80 mm
- net /HSE_IN: track 0.00 -> 8.74 mm
- net +3.3VA: track 0.00 -> 6.99 mm
- net /HSE_OUT: track 0.00 -> 6.37 mm
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- added copper zone on F.Cu, net +3V3
- added copper zone on B.Cu, net GND
- added copper zone on F.Cu, net GND
- added copper zone on F.Cu, net VBUS
Other:
- board text added: "0"
- board text added: "1"
- board text added: "BOOT"
- board text added: "GND"
- board text added: "I2C"
- board text added: "Rx"
- board text added: "SCL"
- board text added: "SDA"
- board text added: "SWCLK"
- board text added: "SWD"
- board text added: "SWDIO"
- board text added: "Tx"
- board text added: "UART"
- board text added: "USB"
- board text added: "v0.1"

Commit message: user logo added to PCB
Parts:
- added G***: LOGO, user_logos:lemonic_logo_20x8mm, B.Cu at (149.7, 81.1)
Other:
- board text added: "STM32F103C6"
